Commit message: tung dag

File: description/robot_core.xacro (robot description, xacro)
@@ -19,5 +19,5 @@
   <link name="base_footprint">
    <visual>
-      <origin xyz="0 0 0" rpy="0 0 0" />
+      <origin xyz="0 0 0" rpy="${pi/2} 0 0" />
       <geometry>
         <box size="0.001 0.001 0.001" />

Commit message: force1

File: description/robot_core.xacro (robot description, xacro)
@@ -19,5 +19,5 @@
   <link name="base_footprint">
    <visual>
-      <origin xyz="0 0 0" rpy="${pi/2} 0 0" />
+      <origin xyz="0 0 0" rpy="0 0 0" />
       <geometry>
         <box size="0.001 0.001 0.001" />
@@ -51,12 +51,3 @@
     </collision>
   </link>
-  <gazebo>
-    <plugin name="object_controller" filename="libgazebo_ros_planar_move.so">
-      <commandTopic>cmd_vel</commandTopic>
-      <odometryTopic>odom</odometryTopic>
-      <odometryFrame>odom</odometryFrame>
-      <odometryRate>20.0</odometryRate>
-      <robotBaseFrame>base_footprint</robotBaseFrame>
-    </plugin>
-  </gazebo>
 </robot>
