Commit message: andre commit

File: description/camera.xacro (robot description, xacro)
@@ -4,9 +4,5 @@
         <parent link="base_link"/>
         <child link="camera_link"/>
-<<<<<<< HEAD
         <origin xyz="0 0 -0.25" rpy="0 ${pi/2} 0"/>
-=======
-        <origin xyz="0 0 -0.05" rpy="0 ${pi/2} 0"/>
->>>>>>> 7589063c09b2835a1d0423d5874da9fdcb3b7831
     </joint>
     <link name="camera_link">

File: description/lidar.xacro (robot description, xacro)
@@ -4,9 +4,5 @@
         <parent link="base_link"/>
         <child link="laser_frame"/>
-<<<<<<< HEAD
         <origin xyz="0 0 0" rpy="0 0 0"/>
-=======
-        <origin xyz="0 0 -2" rpy="0 0 0"/>
->>>>>>> 7589063c09b2835a1d0423d5874da9fdcb3b7831
     </joint>
     <link name="laser_frame">
@@ -41,9 +37,5 @@
                 <range>
                     <min>0.3</min>
-<<<<<<< HEAD
                     <max>20</max>
-=======
-                    <max>5</max>
->>>>>>> 7589063c09b2835a1d0423d5874da9fdcb3b7831
                 </range>
             </ray>

File: description/robot.urdf.xacro (robot description, xacro)
@@ -4,4 +4,3 @@
     <xacro:include filename="robot_core.xacro" />
     <xacro:include filename="camera.xacro" />
-    <xacro:include filename="lidar.xacro" />
 </robot>

File: description/robot_core.xacro (robot description, xacro)
@@ -33,8 +33,4 @@
   <link name="base_link">
     <inertial>
-<<<<<<< HEAD
-=======
-        <origin xyz="0 0 0" />
->>>>>>> 7589063c09b2835a1d0423d5874da9fdcb3b7831
       <mass value="50" />
       <origin xyz="0 0 0" />
@@ -45,5 +41,4 @@
     <visual>
       <geometry>
-<<<<<<< HEAD
         <box size="0.5 0.5 0.5" /> <!-- does not need to match collision -->
       </geometry>
@@ -53,13 +48,4 @@
       <geometry>
         <box size="0.5 0.5 0.5" />
-=======
-        <box size="0.1 0.1 0.1" /> <!-- does not need to match collision -->
-      </geometry>
-    </visual>
-    <collision>
-    <origin xyz="0 0 0" />
-      <geometry>
-        <box size="0.1 0.1 0.1" />
->>>>>>> 7589063c09b2835a1d0423d5874da9fdcb3b7831
       </geometry>
     </collision>

Commit message: I got 2 cams

File: description/camera.xacro (robot description, xacro)
@@ -32,7 +32,7 @@
             <pose> 0 0 0 0 0 0 </pose>
             <visualize>true</visualize>
-            <update_rate>3</update_rate>
+            <update_rate>4</update_rate>
             <camera>
-                <horizontal_fov>1.2</horizontal_fov>
+                <horizontal_fov>2.61799</horizontal_fov>
                 <image>
                     <format>R8G8B8</format>
@@ -41,6 +41,6 @@
                 </image>
                 <clip>
-                    <near>0.5</near>
-                    <far>4.0</far>
+                    <near>0.1</near>
+                    <far>10</far>
                 </clip>
             </camera>

File: description/robot.urdf.xacro (robot description, xacro)
@@ -4,3 +4,4 @@
     <xacro:include filename="robot_core.xacro" />
     <xacro:include filename="camera.xacro" />
+    <xacro:include filename="camera2.xacro" />
 </robot>

File: description/robot_core.xacro (robot description, xacro)
@@ -26,5 +26,5 @@
   </link>
   <joint name="base_link_joint" type="fixed">
-    <origin xyz="0 0 2" rpy="0 0 0" />
+    <origin xyz="0 0 0" rpy="0 0 0" />
     <parent link="base_footprint"/>
     <child link="base_link" />
